Commit message: feat(motion-planner): cartesian trajectory planner with slerp rotation, discontinuity-free phases
Replace SDF-based optimizer with constant-speed cartesian segment planner:
- Slerp rotation interpolation between phase orientations prevents wrist flips
- Rotation-only phases at pre-grasp (1b) and above-home (5b) for smooth transitions
- Keypoint density 2mm with ≥3 waypoints per keypoint for joint-space smoothing
- Staging waypoints route around center pole between arms
- Discontinuity detection (>0.1 rad) with trajectory dump to /tmp

Also includes:
- grasp_selector: graceful fallback with status messages when place target fails
- grasp_selector: SKIP_VLM_RATING mode for geometric-only candidate selection
- dora-pyrealsense: xoq-realsense relay mode for remote camera streaming
- dora-xoq-chat: chat orchestrator for pick-and-place commands
- compiled_fk: pre-baked FK for left arm (~8% faster)
- grasp_trajectory: standalone pick-and-place trajectory generation
- trajectory_json: v3 format with gripper frames

Co-Authored-By: Claude Opus 4.6 <noreply@anthropic.com>

File: examples/openarm/openarm_v10.urdf (robot description, URDF)
Before this commit: robot openarm, 28 links, 27 joints
Joints:
- joint L_J3: origin xyz=0.0301 0.0 0.06625 rpy=0 0 0 -> xyz=0.0301 0.0 0.11625 rpy=0 0 0
- joint R_J3: origin xyz=0.0301 0.0 0.06625 rpy=0 0 0 -> xyz=0.0301 0.0 0.11625 rpy=0 0 0
